Commit message: updated vehicle.xacro file for the pacifica

File: pacifica_vehicle_description/urdf/vehicle.xacro (robot description, xacro)
@@ -7,7 +7,7 @@
     <!-- <xacro:include filename="$(find pacifica_vehicle_description)/urdf/pacifica_18_structure.urdf.xacro" /> -->
 <!-- </robot> -->
-<robot name="pacifica_structure" xmlns:xacro="http://www.ros.org/wiki/xacro" >
+<!-- <robot name="pacifica_structure" xmlns:xacro="http://www.ros.org/wiki/xacro" >
   <xacro:arg name="dae_file" default="$(find dbw_fca_description)/meshes/pacifica_18/body.dae"/>
-  <!-- load parameter -->
+  load parameter
   <xacro:property name="vehicle_info" value="${xacro.load_yaml('$(find pacifica_vehicle_description)/config/vehicle_info.param.yaml')}"/>
   <xacro:property name="half_track_width" value="0.77" />
@@ -88,12 +88,8 @@
     </joint>
   </xacro:macro>
-  <link name="base_footprint" >
-    <visual>
-      <origin xyz="${vehicle_info['/**']['ros__parameters']['wheel_base']/2.0} 0 0" rpy="${pi/2.0} 0 ${pi}"/>
-    </visual>
-  </link>
+  <link name="base_footprint" />
   <link name="base_link" >
     <visual>
-      <origin xyz="-0.06 0 0.1" rpy="0 0 0" />
+      <origin xyz="1.54 0 -0.1825" rpy="0 0 0" />
       <geometry>
         <mesh filename="file://$(arg dae_file)" scale="0.96 0.96 0.96" />
@@ -101,5 +97,5 @@
     </visual>
     <collision>
-      <origin xyz="-0.06 0 0.1" rpy="0 0 0" />
+      <origin xyz="1.54 0 -0.1825" rpy="0 0 0" />
       <geometry>
         <mesh filename="package://dbw_fca_description/meshes/pacifica_18/body_collision.stl" scale="0.96 0.96 0.96" />
@@ -136,10 +132,10 @@
     <parent link="base_link" />
     <child link="hood_logo" />
-    <origin xyz="0 0 0" rpy="0 0 0" />
+    <origin xyz="1.54 0 0" rpy="0 0 0" />
   </joint>
   <joint name="door_logo_joint" type="fixed" >
     <parent link="base_link" />
     <child link="door_logo" />
-    <origin xyz="0 0 0" rpy="0 0 0" />
+    <origin xyz="1.54 0 0" rpy="0 0 0" />
   </joint>
   <xacro:rear_wheel name="rl" x="${-half_wheelbase}" y="${half_track_width}" z="0" flip="0" />
@@ -157,3 +153,16 @@
     </visual>
   </gazebo>
+</robot> -->
+<robot xmlns:xacro="http://ros.org/wiki/xacro">
+  <!-- load parameter -->
+  <xacro:property name="vehicle_info" value="${xacro.load_yaml('$(find pacifica_vehicle_description)/config/vehicle_info.param.yaml')}"/>
+  <!-- vehicle body -->
+  <link name="base_link">
+    <visual>
+      <origin xyz="${vehicle_info['/**']['ros__parameters']['wheel_base']/2.0} 0 ${vehicle_info['/**']['ros__parameters']['wheel_radius']/2.0}" rpy="0 0 0"/>
+      <geometry>
+        <mesh filename="package://pacifica_vehicle_description/mesh/body.dae" scale="1 1 1" rpy="0 0 0"/>
+      </geometry>
+    </visual>
+  </link>
 </robot>

Commit message: updated vehicle_interface.launch to include beliv_vehicle_interface and updated mesh z origin in vehicle.xacro

File: pacifica_vehicle_description/urdf/vehicle.xacro (robot description, xacro)
@@ -162,5 +162,5 @@
       <origin xyz="${vehicle_info['/**']['ros__parameters']['wheel_base']/2.0} 0 ${vehicle_info['/**']['ros__parameters']['wheel_radius']/2.0}" rpy="0 0 0"/>
       <geometry>
-        <mesh filename="package://pacifica_vehicle_description/mesh/body.dae" scale="1 1 1" rpy="0 0 0"/>
+        <mesh filename="package://pacifica_vehicle_description/mesh/body.dae" scale="1 1 1" xyz="0 0 $vehicle_info['/**']['ros__parameters']['wheel_radius']/2.0" rpy="0 0 0"/>
       </geometry>
     </visual>

Commit message: added additional meshes to vehicle.xacro

File: pacifica_vehicle_description/urdf/vehicle.xacro (robot description, xacro)
@@ -1,157 +1,3 @@
 <?xml version="1.0"?>
-<!-- <?xml version="1.0"?>
-<robot xmlns:xacro="http://ros.org/wiki/xacro"> -->
-  <!-- load parameter -->
-  <!-- <xacro:property name="vehicle_info" value="${xacro.load_yaml('$(find pacifica_vehicle_description)/config/vehicle_info.param.yaml')}"/> -->
-  <!-- vehicle body -->
-    <!-- <xacro:include filename="$(find pacifica_vehicle_description)/urdf/pacifica_18_structure.urdf.xacro" /> -->
-<!-- </robot> -->
-<!-- <robot name="pacifica_structure" xmlns:xacro="http://www.ros.org/wiki/xacro" >
-  <xacro:arg name="dae_file" default="$(find dbw_fca_description)/meshes/pacifica_18/body.dae"/>
-  load parameter
-  <xacro:property name="vehicle_info" value="${xacro.load_yaml('$(find pacifica_vehicle_description)/config/vehicle_info.param.yaml')}"/>
-  <xacro:property name="half_track_width" value="0.77" />
-  <xacro:property name="half_wheelbase" value="1.54" />
-  <xacro:property name="wheel_radius" value="0.365" />
-  <xacro:property name="wheel_thickness" value="0.25" />
-  <xacro:property name="wheel_mass" value="10.0" />
-  <xacro:property name="body_mass" value="2242.0" />
-  <xacro:property name="body_width" value="${2*half_track_width}" />
-  <xacro:property name="body_depth" value="${2*half_wheelbase + 1.2}" />
-  <xacro:property name="body_length" value="0.6" />
-  <xacro:macro name="rear_wheel" params="name x y z flip" >
-    <link name="wheel_${name}" >
-      <visual>
-        <origin xyz="0 0 0" rpy="1.57079632679 ${flip * 3.1415926535} 0" />
-        <geometry>
-          <mesh filename="package://dbw_fca_description/meshes/pacifica_18/wheel.dae" />
-        </geometry>
-      </visual>
-      <collision>
-        <geometry>
-          <cylinder radius="${wheel_radius}" length="${wheel_thickness}" />
-        </geometry>
-      </collision>
-      <inertial>
-        <origin xyz="0 0 0" rpy="0 0 0"/>
-        <mass value="1.0"/>
-        <inertia ixx="1.0" ixy="0" ixz="0" iyy="1.0" iyz="0" izz="1.0"/>
-      </inertial>
-    </link>
-    <joint name="wheel_${name}_joint" type="continuous" >
-      <parent link="base_link" />
-      <child link="wheel_${name}" />
-      <origin xyz="${x} ${y} ${z}" rpy="-1.57079632679 0 0" />
-      <axis xyz="0 0 1" />
-      <limit effort="0" velocity="22.0" />
-    </joint>
-  </xacro:macro>
-  <xacro:macro name="front_wheel" params="name x y z flip" >
-    <link name="wheel_${name}" >
-      <visual>
-        <origin xyz="0 0 0" rpy="1.57079632679 ${flip * pi} 0" />
-        <geometry>
-          <mesh filename="package://dbw_fca_description/meshes/pacifica_18/wheel.dae" />
-        </geometry>
-      </visual>
-      <collision>
-        <geometry>
-          <cylinder radius="${wheel_radius}" length="${wheel_thickness}" />
-        </geometry>
-      </collision>
-      <inertial>
-        <origin xyz="0 0 0" rpy="0 0 0"/>
-        <mass value="${wheel_mass}"/>
-        <inertia ixx="${wheel_mass/12*(3*wheel_radius*wheel_radius + wheel_thickness*wheel_thickness)}" ixy="0" ixz="0" iyy="${wheel_mass/12*(3*wheel_radius*wheel_radius + wheel_thickness*wheel_thickness)}" iyz="0" izz="${wheel_mass/2 * wheel_radius*wheel_radius}"/>
-      </inertial>
-    </link>
-    <link name="steer_${name}" >
-      <inertial>
-        <origin xyz="-0.013054 -0.0295 0" rpy="0 0 0"/>
-        <mass value="1.0"/>
-        <inertia ixx="0.037227" ixy="0" ixz="0" iyy="0.04" iyz="0" izz="0.06"/>
-      </inertial>
-    </link>
-    <joint name="steer_${name}_joint" type="revolute" >
-      <parent link="base_link" />
-      <child link="steer_${name}" />
-      <origin xyz="${x} ${y} ${z}" rpy="0 0 0" />
-      <axis xyz="0 0 1" />
-      <limit upper="0.6" lower="-0.6" effort="0.0" velocity="0.0" />
-    </joint>
-    <joint name="wheel_${name}_joint" type="continuous" >
-      <parent link="steer_${name}" />
-      <child link="wheel_${name}" />
-      <origin xyz="0 0 0" rpy="-1.57079632679 0 0" />
-      <axis xyz="0 0 1" />
-      <limit effort="0" velocity="22.0" />
-    </joint>
-  </xacro:macro>
-  <link name="base_footprint" />
-  <link name="base_link" >
-    <visual>
-      <origin xyz="1.54 0 -0.1825" rpy="0 0 0" />
-      <geometry>
-        <mesh filename="file://$(arg dae_file)" scale="0.96 0.96 0.96" />
-      </geometry>
-    </visual>
-    <collision>
-      <origin xyz="1.54 0 -0.1825" rpy="0 0 0" />
-      <geometry>
-        <mesh filename="package://dbw_fca_description/meshes/pacifica_18/body_collision.stl" scale="0.96 0.96 0.96" />
-      </geometry>
-      </collision>
-    <inertial>
-      <origin xyz="-0.25 0 0.3" rpy="0 0 0"/>
-      <mass value="${body_mass}"/>
-      <inertia ixx="${body_mass/12 * (body_width*body_width + body_length*body_length)}" ixy="0" ixz="0" iyy="${body_mass/12 * (body_length*body_length + body_depth*body_depth)}" iyz="0" izz="${body_mass/12 * (body_width*body_width + body_depth*body_depth)}"/>
-    </inertial>
-  </link>
-  <link name="hood_logo" >
-    <visual>
-      <origin xyz="-0.06 0 0.102" rpy="0 0 0" />
-      <geometry>
-        <mesh filename="package://dbw_fca_description/meshes/pacifica_18/hood_logo.dae" scale="0.96 0.96 0.96" />
-      </geometry>
-    </visual>
-  </link>
-  <link name="door_logo" >
-    <visual>
-      <origin xyz="-0.06 0 0.102" rpy="0 0 0" />
-      <geometry>
-        <mesh filename="package://dbw_fca_description/meshes/pacifica_18/door_logo.dae" scale="0.965 0.965 0.965" />
-      </geometry>
-    </visual>
-  </link>
-  <joint name="base_link_joint" type="fixed" >
-    <parent link="base_footprint" />
-    <child link="base_link" />
-    <origin xyz="${half_wheelbase} 0 ${wheel_radius}" rpy="0 0 0" />
-  </joint>
-  <joint name="hood_logo_joint" type="fixed" >
-    <parent link="base_link" />
-    <child link="hood_logo" />
-    <origin xyz="1.54 0 0" rpy="0 0 0" />
-  </joint>
-  <joint name="door_logo_joint" type="fixed" >
-    <parent link="base_link" />
-    <child link="door_logo" />
-    <origin xyz="1.54 0 0" rpy="0 0 0" />
-  </joint>
-  <xacro:rear_wheel name="rl" x="${-half_wheelbase}" y="${half_track_width}" z="0" flip="0" />
-  <xacro:rear_wheel name="rr" x="${-half_wheelbase}" y="${-half_track_width}" z="0" flip="1" />
-  <xacro:front_wheel name="fl" x="${half_wheelbase}" y="${half_track_width}" z="0" flip="0" />
-  <xacro:front_wheel name="fr" x="${half_wheelbase}" y="${-half_track_width}" z="0" flip="1" />
-  <gazebo reference="hood_logo" >
-    <visual>
-      <transparency>0.01</transparency>
-    </visual>
-  </gazebo>
-  <gazebo reference="door_logo" >
-    <visual>
-      <transparency>0.01</transparency>
-    </visual>
-  </gazebo>
-</robot> -->
 <robot xmlns:xacro="http://ros.org/wiki/xacro">
   <!-- load parameter -->
@@ -159,8 +5,51 @@
   <!-- vehicle body -->
   <link name="base_link">
+    <!-- body -->
     <visual>
-      <origin xyz="${vehicle_info['/**']['ros__parameters']['wheel_base']/2.0} 0 ${vehicle_info['/**']['ros__parameters']['wheel_radius']/2.0}" rpy="0 0 0"/>
+      <origin xyz="${vehicle_info['/**']['ros__parameters']['wheel_base']/2.0} 0 ${vehicle_info['/**']['ros__parameters']['wheel_radius']}" rpy="0 0 0" />
       <geometry>
-        <mesh filename="package://pacifica_vehicle_description/mesh/body.dae" scale="1 1 1" xyz="0 0 $vehicle_info['/**']['ros__parameters']['wheel_radius']/2.0" rpy="0 0 0"/>
+        <mesh filename="package://pacifica_vehicle_description/mesh/body.dae" scale="0.96 0.96 0.96" />
+      </geometry>
+    </visual>
+    <!-- rearwheel 1 -->
+    <visual>
+      <origin xyz="0 ${vehicle_info['/**']['ros__parameters']['wheel_tread']/2.0} ${vehicle_info['/**']['ros__parameters']['wheel_radius']}" rpy="0 3.1415926535 0" />
+      <geometry>
+        <mesh filename="package://pacifica_vehicle_description/mesh/wheel.dae" scale="1 1 1" />
+      </geometry>
+    </visual>
+    <!-- rear wheel 2 -->
+    <visual>
+      <origin xyz="0 ${vehicle_info['/**']['ros__parameters']['wheel_tread']/-2.0} ${vehicle_info['/**']['ros__parameters']['wheel_radius']}" rpy="0 3.1415926535 3.1415926535" />
+      <geometry>
+        <mesh filename="package://pacifica_vehicle_description/mesh/wheel.dae" scale="1 1 1" />
+      </geometry>
+    </visual>
+    <!-- front wheel 1 -->
+    <visual>
+      <origin xyz="${vehicle_info['/**']['ros__parameters']['wheel_base']/1.0} ${vehicle_info['/**']['ros__parameters']['wheel_tread']/2.0} ${vehicle_info['/**']['ros__parameters']['wheel_radius']}" rpy="0 3.1415926535 0" />
+      <geometry>
+        <mesh filename="package://pacifica_vehicle_description/mesh/wheel.dae" scale="1 1 1" />
+      </geometry>
+    </visual>
+    <!-- front wheel 2 -->
+    <visual>
+      <origin xyz="${vehicle_info['/**']['ros__parameters']['wheel_base']/1.0} ${vehicle_info['/**']['ros__parameters']['wheel_tread']/-2.0} ${vehicle_info['/**']['ros__parameters']['wheel_radius']}" rpy="0 3.1415926535 3.1415926535" />
+      <geometry>
+        <mesh filename="package://pacifica_vehicle_description/mesh/wheel.dae" scale="1 1 1" />
+      </geometry>
+    </visual>
+    <!-- hood logo -->
+    <visual>
+      <origin xyz="${vehicle_info['/**']['ros__parameters']['wheel_base']/2.0} 0 ${vehicle_info['/**']['ros__parameters']['wheel_radius']}" rpy="0 0 0" />
+      <geometry>
+        <mesh filename="package://pacifica_vehicle_description/mesh/hood_logo.dae" scale="0.96 0.96 0.96" />
+      </geometry>
+    </visual>
+    <!-- door logo -->
+    <visual>
+      <origin xyz="${vehicle_info['/**']['ros__parameters']['wheel_base']/2.0} 0 ${vehicle_info['/**']['ros__parameters']['wheel_radius']}" rpy="0 0 0" />
+      <geometry>
+        <mesh filename="package://pacifica_vehicle_description/mesh/door_logo.dae" scale="0.965 0.965 0.965" />
       </geometry>
     </visual>
